File: dap-link.kicad_pcb (KiCad board)
At the start: 4 copper layers, 75 x 30 mm, 53 parts, among them J1 Molex 0473460001, J2 SWD 6 PIN 2.54mm, J3 JTAG/SWD 10 pin 2.54mm, J4 JTAG/SWD 10 pin 1.27mm, J5 JTAG/SWD 20 PIN 1.27mm, J6 DAPLink Flash, Q1 MMBT3904, U1 SC573V33RTRC, U2 STM32F103CBTx, U3 150141SV73110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

Commit message: case v1
Parts:
- removed D5, D6: HSP051-4N10, MyLib:UQFN1.9x1_10L
- removed J5: JTAG/SWD 20 PIN 1.27mm, Connector_PinHeader_1.27mm:PinHeader_2x10_P1.27mm_Vertical_SMD
- removed J6: DAPLink Flash, MyLib:PinHeader_2x05_P1.27mm_Vertical_SMD
- removed R16, R17: 22R, Resistor_SMD:R_0603_1608Metric
- removed R6: 10k, Resistor_SMD:R_0603_1608Metric
- J2: value SWD 6 PIN 2.54mm -> Conn_01x05_Male; footprint Connector_PinHeader_2.54mm:PinHeader_1x06_P2.54mm_Vertical -> MyLib:SWD_SOLDER
- J3: value JTAG/SWD 10 pin 2.54mm -> SWD 10 pin 2.54mm
- J4: value JTAG/SWD 10 pin 1.27mm -> SWD 10 pin 1.27mm
- Y1: footprint Crystal:Crystal_SMD_HC49-SD -> MyLib:ECS-023G
- moved J2 45.0 mm to (85.6, 65.1), turned to -90 degrees
- moved U3 26.6 mm to (73.0, 66.0), turned to -90 degrees
- moved R2 21.4 mm to (73.0, 69.6), turned to 180 degrees
- moved R10 18.3 mm to (76.5, 66.5), turned to 90 degrees
- moved R5 14.7 mm to (84.5, 82.7)
- moved R19 14.3 mm to (94.9, 68.6), turned to 90 degrees
- moved R20 14.0 mm to (94.9, 71.9)
- moved J4 12.5 mm to (51.0, 76.0)
- moved R13 11.4 mm to (91.6, 81.0)
- moved H3 10.0 mm to (47.0, 87.0)
- moved H4 10.0 mm to (47.0, 65.0)
- moved R21 9.06 mm to (92.3, 69.4), turned to 0 degrees
- moved C10 8.95 mm to (93.8, 80.4), turned to 90 degrees
- moved D7 8.43 mm to (73.9, 85.5), turned to 90 degrees
- moved C1 7.65 mm to (79.1, 65.5), turned to -90 degrees
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Connections:
- net Net-(R4-Pad2) renamed /BOOT0
- D7 pad 1: SWO -> VTREF
- D7 pad 2: TCLK -> SWCLK
- D7 pad 3: TDI -> SWDIO
- J2 pad 1: VTREF -> +3V3
- J2 pad 2: TCLK -> STM_SWDIO
- J2 pad 3: GND -> STM_SWCLK
- J2 pad 4: TMS -> STM_NRST
- J2 pad 5: NRST -> GND
- J3 pad 2: TMS -> SWDIO
- J3 pad 4: TCLK -> SWCLK
- J3 pad 6: SWO -> unconnected-(J3-Pad6)
- J3 pad 8: TDI -> unconnected-(J3-Pad8)
- J4 pad 2: TMS -> SWDIO
- J4 pad 4: TCLK -> SWCLK
- J4 pad 6: SWO -> unconnected-(J4-Pad6)
- J4 pad 8: TDI -> unconnected-(J4-Pad8)
- R10 pad 1: /LED -> /CONNECTED_LED
- R13 pad 1: TCLK -> SWCLK
- R13 pad 2: /T_JTCK -> /T_SWCLK
- R14 pad 1: TMS -> SWDIO
- R14 pad 2: /T_JTMS -> /T_SWDIO_IN
- R2 pad 1: /LED -> /COM_LED
- R3 pad 1: /T_SWDIO_IN -> /T_SWDIO_OUT
- R3 pad 2: /T_JTMS -> /T_SWDIO_IN
- R5 pad 1: Net-(R5-Pad1) -> GND
- R5 pad 2: GND -> /BOOT1
- U2 pad 15: /T_JTCK -> unconnected-(U2-Pad15)
- U2 pad 16: /T_JTDO -> unconnected-(U2-Pad16)
- U2 pad 17: /T_JTDI -> unconnected-(U2-Pad17)
- U2 pad 2: Net-(R5-Pad1) -> unconnected-(U2-Pad2)
- U2 pad 20: GND -> /BOOT1
- U2 pad 25: /T_JTMS -> /T_SWDIO_IN
- U2 pad 26: /T_JTCK -> /T_SWCLK
- U2 pad 27: /T_SWDIO_IN -> /T_SWDIO_OUT
- U2 pad 28: GND -> /POWER_EN_LED
- U2 pad 29: GND -> /CONNECTED_LED
- U2 pad 3: Net-(R6-Pad1) -> unconnected-(U2-Pad3)
- U2 pad 30: /LED -> /COM_LED
- U2 pad 31: /T_SWO -> unconnected-(U2-Pad31)
- U2 pad 39: +3V3 -> unconnected-(U2-Pad39)
Routing:
- net TMS: track 87.3 -> 0.00 mm, vias 5 -> 0
- net TCLK: track 71.1 -> 0.00 mm, vias 5 -> 0
- net SWO: track 65.3 -> 0.00 mm, vias 3 -> 0
- net TDI: track 63.4 -> 0.00 mm, vias 2 -> 0
- net SWDIO: track 0.00 -> 51.2 mm
- net SWCLK: track 0.00 -> 49.7 mm
- net VTREF: track 108.9 -> 71.9 mm, vias 5 -> 6
- net NRST: track 62.2 -> 32.8 mm
- net Net-(Q1-Pad1): track 24.6 -> 5.87 mm
- net /COM_LED: track 0.00 -> 18.0 mm, vias 0 -> 2
- net /CONNECTED_LED: track 0.00 -> 16.7 mm, vias 0 -> 2
- net STM_NRST: track 35.5 -> 20.7 mm
- net /T_SWO: track 13.7 -> 0.00 mm
- net /T_JTCK: track 11.1 -> 0.00 mm
- net Net-(D1-Pad1): track 2.66 -> 9.22 mm, vias 0 -> 2
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- added copper zone on B.Cu, net VTREF
- added copper zone on F.Cu, net VTREF
Other:
- board size 75 x 30 mm -> 65 x 30 mm

Commit message: changes
Parts:
- removed U3: 150141SV73110, MyLib:150141SV73110
- added D5: 150141SV73110, MyLib:150141SV73110, F.Cu at (73.0, 66.1)
- added J5: TC2050-IDC, MyLib:TAG-CONNECT_TC2050-IDC, F.Cu at (93.0, 65.6)
- C2, C3: value 20p -> 18p
- D1, D2, D3: value D_Small -> SM5817PL-TP; footprint Diode_SMD:Nexperia_CFP3_SOD-123W -> Diode_SMD:D_SOD-123
- moved J2 5.17 mm to (81.3, 62.2)
- moved J3 2.24 mm to (62.5, 75.0)
- moved J4 2.24 mm to (53.0, 75.0)
- moved R21 2.20 mm to (92.2, 71.6), turned to -90 degrees
- moved R19 1.95 mm to (94.5, 70.5), turned to 180 degrees
- moved R20 1.50 mm to (94.5, 73.3), turned to 0 degrees
- moved D4 1.00 mm to (100.9, 75.9)
- moved H1 1.00 mm to (104.0, 64.0)
- moved H2 1.00 mm to (104.0, 86.0)
- moved H3 1.00 mm to (47.0, 86.0)
- moved H4 1.00 mm to (47.0, 64.0)
- moved J1 1.00 mm to (106.5, 75.0)
- moved R18 1.00 mm to (100.7, 72.7)
- moved R12 0.95 mm to (76.6, 87.4)
- moved D1 0.94 mm to (70.3, 87.5)
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Connections:
- net Net-(D1-Pad1) renamed /T_VTREF
- U2 pad 29: /CONNECTED_LED -> unconnected-(U2-Pad29)
- U2 pad 42: unconnected-(U2-Pad42) -> /CONNECTED_LED
Routing:
- net STM_NRST: track 20.7 -> 41.2 mm
- net STM_SWCLK: track 10.1 -> 26.2 mm, vias 2 -> 0
- net VTREF: track 71.9 -> 57.9 mm
- net GND: track 30.9 -> 44.5 mm, vias 49 -> 105
- net STM_SWDIO: track 10.1 -> 20.1 mm, vias 2 -> 3
- net +3V3: track 30.0 -> 37.3 mm
- net /CONNECTED_LED: track 16.7 -> 13.5 mm
- net Net-(Q1-Pad1): track 5.87 -> 7.97 mm
- net SWCLK: track 49.7 -> 51.1 mm
- net NRST: track 32.8 -> 31.5 mm
- net SWDIO: track 51.2 -> 50.1 mm
- net /USB_RENUMn: track 6.61 -> 7.56 mm
- net Net-(Q1-Pad2): track 2.20 -> 3.01 mm
- net Net-(D3-Pad1): track 8.45 -> 7.81 mm
- net /USB_DP: track 18.2 -> 17.6 mm
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Other:
- board text added: "1 2 3 4 5 6 7 8 9 10"
- board text added: "10 PIN SWD OUT (J3, J4)"
- board text added: "3V3"
- board text added: "5V"
- board text added: "NAME SWDIO SWCLK NC NC NRST"
- board text added: "PINOUT J2 1 3V3 2 SWDIO 3 SWCLK 4 NRST 5 GND"
- board text added: "PINOUT J5 3V3 SWDIO GND SWCLK GND NC GND NC GND NRST"
- board text added: "SET JP1 ON FRONT SIDE TO FORCE VTREF TO 3.3V OR 5V"
- board text added: "USE J2 OR J5 TO FLASH BOOTLOADER"
- board text removed: "10 PIN CONNECTOR PINOUT"
- board text removed: "20 PIN CONNECTOR PINOUT"
- board text removed: "6 PIN SWD"
- board text removed: "GND"
- board text removed: "Jumpers not set -> VTREF = VDUT Pos 1 set -> VTREF = 3V3 Pos 2 set -> VTREF = 5V"
- board text removed: "NAME SWDIO/TMS SWCLK/TCLK SWO TDI NRST"
- board text removed: "NAME VTREF GND GND GND GND GND GND GND GND GND"
- board text removed: "NAME VTREF NC TDI SWDIO/TMS SWCLK/TCLK NC SWO NRST NC NC"
- board text removed: "NR 1 3 5 7 9 11 13 15 17 19"
- board text removed: "NR 2 4 6 8 10 12 14 16 18 20"
- board text removed: "NRST"
- board text removed: "SWCLK"
- board text removed: "SWDIO"
- board text removed: "SWO"
- board text removed: "VTREF"

Commit message: changed 1.27mm swd out connector to horizontal orientation
Parts:
- J4: value SWD 10 pin 1.27mm -> SWD 10 pin 2.54mm; footprint MyLib:PinHeader_2x05_P1.27mm_Vertical_SMD -> MyLib:GBED204-0579B001C1AD
- moved H3 5.50 mm to (52.5, 86.0)
- moved H4 5.50 mm to (52.5, 64.0)
- moved J4 2.30 mm to (55.3, 75.0), turned to -90 degrees
Connections:
- U2 pad 28: /POWER_EN_LED -> unconnected-(U2-Pad28)
Routing:
- net GND: track 44.5 -> 36.3 mm, vias 105 -> 56
- net VTREF: track 57.9 -> 54.4 mm
- net SWDIO: track 50.1 -> 47.5 mm
- net SWCLK: track 51.1 -> 48.9 mm
- net NRST: track 31.5 -> 29.7 mm
Other:
- board size 65 x 30 mm -> 59.5 x 30 mm
- board text removed: "1 2 3 4 5 6 7 8 9 10"
